Commit message: Completed tutorial.

File: src/robot_description/urdf/robot.urdf (robot description, URDF)
Before this commit: robot robot1, 4 links, 3 joints
Links:
- added link wheel_4; visual cylinder length=0.05 radius=0.05
Joints:
- added joint base_to_wheel4: type fixed, parent base_link, child wheel_4, origin xyz=0 0 0
